File: Eagle/Micromouse2/Micromouse2.sch (EAGLE design)
At the start: 11 parts, among them IC1 LMX2322, IC2 LM50

Commit message: update schematic
Connections:
- new net TICK1: JP1.12, JP3.5
- new net TICK2: JP1.11, JP4.5
- net GND: now also JP1.20
- net VCC: now also JP1.19
Other:
- moved on the sheet: JP1
Changed lines of the file:
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@@
 <part name="C3" library="adafruit" deviceset="C-US" device="C0805" value="0.1uF"/>
 <part name="C5" library="adafruit" deviceset="C-US" device="C0805" value=".33uF"/>
+<part name="GND7" library="supply1" deviceset="GND" device=""/>
+<part name="P+7" library="supply1" deviceset="VCC" device=""/>
 </parts>
 <sheets>
@@
 <instance part="C1" gate="G$1" x="55.88" y="106.68"/>
 <instance part="C2" gate="G$1" x="58.42" y="63.5"/>
-<instance part="JP1" gate="A" x="-35.56" y="66.04" rot="R180"/>
+<instance part="JP1" gate="A" x="-43.18" y="66.04" rot="R180"/>
 <instance part="JP2" gate="A" x="109.22" y="66.04"/>
 <instance part="JP3" gate="A" x="2.54" y="147.32" rot="MR90"/>
@@
 <instance part="C3" gate="G$1" x="27.94" y="137.16"/>
 <instance part="C5" gate="G$1" x="22.86" y="160.02"/>
+<instance part="GND7" gate="1" x="-17.78" y="58.42"/>
+<instance part="P+7" gate="VCC" x="-25.4" y="104.14"/>
 </instances>
 <busses>
@@
 <junction x="22.86" y="132.08"/>
 </segment>
+<segment>
+<pinref part="JP1" gate="A" pin="20"/>
+<wire x1="-40.64" y1="91.44" x2="-17.78" y2="91.44" width="0.1524" layer="91"/>
+<wire x1="-17.78" y1="91.44" x2="-17.78" y2="60.96" width="0.1524" layer="91"/>
+<pinref part="GND7" gate="1" pin="GND"/>
+</segment>
 </net>
 <net name="VCC" class="0">
@@
 <junction x="35.56" y="165.1"/>
 </segment>
+<segment>
+<pinref part="JP1" gate="A" pin="19"/>
+<wire x1="-40.64" y1="88.9" x2="-25.4" y2="88.9" width="0.1524" layer="91"/>
+<wire x1="-25.4" y1="88.9" x2="-25.4" y2="101.6" width="0.1524" layer="91"/>
+<pinref part="P+7" gate="VCC" pin="VCC"/>
+</segment>
 </net>
 <net name="N$2" class="0">
@@
 </segment>
 </net>
+<net name="TICK2" class="0">
+<segment>
+<pinref part="JP1" gate="A" pin="11"/>
+<wire x1="-40.64" y1="68.58" x2="-27.94" y2="68.58" width="0.1524" layer="91"/>
+<label x="-27.94" y="68.58" size="1.778" layer="95" xref="yes"/>
+</segment>
+<segment>
+<pinref part="JP4" gate="A" pin="5"/>
+<wire x1="63.5" y1="144.78" x2="63.5" y2="139.7" width="0.1524" layer="91"/>
+<wire x1="63.5" y1="139.7" x2="55.88" y2="139.7" width="0.1524" layer="91"/>
+<label x="55.88" y="139.7" size="1.778" layer="95" rot="R180" xref="yes"/>
+</segment>
+</net>
+<net name="TICK1" class="0">
+<segment>
+<pinref part="JP1" gate="A" pin="12"/>
+<wire x1="-40.64" y1="71.12" x2="-35.56" y2="71.12" width="0.1524" layer="91"/>
+<label x="-35.56" y="71.12" size="1.778" layer="95" xref="yes"/>
+</segment>
+<segment>
+<pinref part="JP3" gate="A" pin="5"/>
+<wire x1="0" y1="144.78" x2="0" y2="137.16" width="0.1524" layer="91"/>
+<wire x1="0" y1="137.16" x2="-20.32" y2="137.16" width="0.1524" layer="91"/>
+<label x="-20.32" y="137.16" size="1.778" layer="95" rot="R180" xref="yes"/>
+</segment>
+</net>

Commit message: Updated Eagle Schematic
Parts:
- added R1, R2, R3, R4: (no value), adafruit:R-US_R0805
- added S1: (no value), adafruit:EG1218S
- added T1, T2: 2N2222, adafruit:2N2222
Connections:
- new net CHECK_EN: JP1.13, T1.B, T2.B
- new net N$10: R2.1, T2.C
- new net N$11: R1.1, R2.2, T1.C
- new net N$7: S1.S
- new net N$8: R4.2, T1.E
- new net N$9: R3.2, T2.E
- net GND: now also R3.1, R4.1
- net VCC: now also R1.2, S1.P
Changed lines of the file:
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@@
 <part name="GND7" library="supply1" deviceset="GND" device=""/>
 <part name="P+7" library="supply1" deviceset="VCC" device=""/>
+<part name="S1" library="adafruit" deviceset="EG1218" device="S"/>
+<part name="P+8" library="supply1" deviceset="VCC" device=""/>
+<part name="T1" library="adafruit" deviceset="2N2222" device=""/>
+<part name="R1" library="adafruit" deviceset="R-US_" device="R0805"/>
+<part name="R2" library="adafruit" deviceset="R-US_" device="R0805"/>
+<part name="GND8" library="supply1" deviceset="GND" device=""/>
+<part name="P+9" library="supply1" deviceset="VCC" device=""/>
+<part name="T2" library="adafruit" deviceset="2N2222" device=""/>
+<part name="R3" library="adafruit" deviceset="R-US_" device="R0805"/>
+<part name="R4" library="adafruit" deviceset="R-US_" device="R0805"/>
+<part name="GND9" library="supply1" deviceset="GND" device=""/>
 </parts>
 <sheets>
@@
 <instance part="GND7" gate="1" x="-17.78" y="58.42"/>
 <instance part="P+7" gate="VCC" x="-25.4" y="104.14"/>
+<instance part="S1" gate="1" x="-60.96" y="162.56" rot="R90"/>
+<instance part="P+8" gate="VCC" x="-48.26" y="165.1" rot="R270"/>
+<instance part="T1" gate="G$1" x="-66.04" y="114.3" rot="MR0"/>
+<instance part="R1" gate="G$1" x="-86.36" y="144.78" rot="R90"/>
+<instance part="R2" gate="G$1" x="-86.36" y="129.54" rot="R90"/>
+<instance part="GND8" gate="1" x="-86.36" y="91.44"/>
+<instance part="P+9" gate="VCC" x="-86.36" y="157.48"/>
+<instance part="T2" gate="G$1" x="-88.9" y="114.3"/>
+<instance part="R3" gate="G$1" x="-86.36" y="101.6" rot="R90"/>
+<instance part="R4" gate="G$1" x="-68.58" y="101.6" rot="R90"/>
+<instance part="GND9" gate="1" x="-83.82" y="165.1"/>
 </instances>
 <busses>
@@
 <pinref part="GND7" gate="1" pin="GND"/>
 </segment>
+<segment>
+<pinref part="R4" gate="G$1" pin="1"/>
+<pinref part="R3" gate="G$1" pin="1"/>
+<wire x1="-68.58" y1="96.52" x2="-86.36" y2="96.52" width="0.1524" layer="91"/>
+<pinref part="GND8" gate="1" pin="GND"/>
+<wire x1="-86.36" y1="93.98" x2="-86.36" y2="96.52" width="0.1524" layer="91"/>
+<junction x="-86.36" y="96.52"/>
+</segment>
+<segment>
+<wire x1="-83.82" y1="177.8" x2="-83.82" y2="167.64" width="0.1524" layer="91"/>
+<pinref part="GND9" gate="1" pin="GND"/>
+</segment>
 </net>
 <net name="VCC" class="0">
@@
 <pinref part="P+7" gate="VCC" pin="VCC"/>
 </segment>
+<segment>
+<pinref part="S1" gate="1" pin="P"/>
+<wire x1="-55.88" y1="165.1" x2="-50.8" y2="165.1" width="0.1524" layer="91"/>
+<pinref part="P+8" gate="VCC" pin="VCC"/>
+</segment>
+<segment>
+<pinref part="R1" gate="G$1" pin="2"/>
+<pinref part="P+9" gate="VCC" pin="VCC"/>
+<wire x1="-86.36" y1="149.86" x2="-86.36" y2="154.94" width="0.1524" layer="91"/>
+</segment>
 </net>
 <net name="N$2" class="0">
@@
 </segment>
 </net>
+<net name="N$8" class="0">
+<segment>
+<pinref part="R4" gate="G$1" pin="2"/>
+<pinref part="T1" gate="G$1" pin="E"/>
+<wire x1="-68.58" y1="106.68" x2="-68.58" y2="109.22" width="0.1524" layer="91"/>
+</segment>
+</net>
+<net name="N$9" class="0">
+<segment>
+<pinref part="R3" gate="G$1" pin="2"/>
+<pinref part="T2" gate="G$1" pin="E"/>
+<wire x1="-86.36" y1="106.68" x2="-86.36" y2="109.22" width="0.1524" layer="91"/>
+</segment>
+</net>
+<net name="N$10" class="0">
+<segment>
+<pinref part="T2" gate="G$1" pin="C"/>
+<pinref part="R2" gate="G$1" pin="1"/>
+<wire x1="-86.36" y1="119.38" x2="-86.36" y2="124.46" width="0.1524" layer="91"/>
+</segment>
+</net>
+<net name="N$11" class="0">
+<segment>
+<pinref part="R2" gate="G$1" pin="2"/>
+<pinref part="R1" gate="G$1" pin="1"/>
+<wire x1="-86.36" y1="134.62" x2="-86.36" y2="137.16" width="0.1524" layer="91"/>
+<pinref part="T1" gate="G$1" pin="C"/>
+<wire x1="-86.36" y1="137.16" x2="-86.36" y2="139.7" width="0.1524" layer="91"/>
+<wire x1="-86.36" y1="137.16" x2="-68.58" y2="137.16" width="0.1524" layer="91"/>
+<wire x1="-68.58" y1="137.16" x2="-68.58" y2="119.38" width="0.1524" layer="91"/>
+<junction x="-86.36" y="137.16"/>
+</segment>
+</net>
+<net name="CHECK_EN" class="0">
+<segment>
+<pinref part="JP1" gate="A" pin="13"/>
+<wire x1="-40.64" y1="73.66" x2="-55.88" y2="73.66" width="0.1524" layer="91"/>
+<label x="-55.88" y="73.66" size="1.778" layer="95" rot="R180" xref="yes"/>
+</segment>
+<segment>
+<pinref part="T2" gate="G$1" pin="B"/>
+<wire x1="-91.44" y1="114.3" x2="-96.52" y2="114.3" width="0.1524" layer="91"/>
+<label x="-96.52" y="114.3" size="1.778" layer="95" rot="R180" xref="yes"/>
+</segment>
+<segment>
+<pinref part="T1" gate="G$1" pin="B"/>
+<wire x1="-63.5" y1="114.3" x2="-60.96" y2="114.3" width="0.1524" layer="91"/>
+<label x="-60.96" y="114.3" size="1.778" layer="95" xref="yes"/>
+</segment>
+</net>
+<net name="N$7" class="0">
+<segment>
+<pinref part="S1" gate="1" pin="S"/>
+<wire x1="-66.04" y1="167.64" x2="-73.66" y2="167.64" width="0.1524" layer="91"/>
+<wire x1="-73.66" y1="167.64" x2="-73.66" y2="177.8" width="0.1524" layer="91"/>
+</segment>
+</net>

Commit message: Update to schematic2
Parts:
- removed R3, R4: (no value), adafruit:R-US_R0805
- removed T1, T2: 2N2222, adafruit:2N2222
Connections:
- removed net N$11: R1.1, R2.2, T1.C
- removed net N$8: R4.2, T1.E
- removed net N$9: R3.2, T2.E
- new net +3V3: JP2.1, JP3.4, JP4.4
- new net BATT_CHECK: JP1.7, R1.1, R2.2
- net +5V: now also C1.1, C4.1, IC1.CE; no longer JP3.4, JP4.4
- net CHECK_EN: no longer T1.B, T2.B
- net GND: now also IC1.GND, IC1.VP; no longer R3.1, R4.1
- net N$10: no longer T2.C
- net VCC: no longer C1.1, C4.1, IC1.CE

Commit message: Updating schematic and adding board
Parts:
- removed C3: 0.1uF, adafruit:C-USC0805
- removed C5: .33uF, adafruit:C-USC0805
- removed IC2: LM50, linear:LM50
- added BATT: (no value), adafruit:JST_2PIN-THM
- added JUMPER: (no value), pinhead:PINHD-2X4
- added S2: (no value), adafruit:EG1218S
- renumbered IC1 to DRIVER, JP1 to RIGHT, JP2 to LEFT, JP3 to RM, JP4 to LM
Connections:
- removed net +5V: C1.1, C3.1, C4.1, DRIVER.CE, IC2.VO
- removed net N$10: R2.1
- new net FSENS_EN: JUMPER.6, LEFT.12
- new net LF_SENS: JUMPER.4, RIGHT.1
- new net LS_SENS: JUMPER.7, RIGHT.3
- new net N$8: DRIVER.FIN, RIGHT.9
- new net N$9: DRIVER.OSCIN, RIGHT.10
- new net RF_SENS: JUMPER.2, RIGHT.2
- new net RS_SENS: JUMPER.5, RIGHT.4
- new net SSENS_EN: JUMPER.3, LEFT.11
- new net VDD: RIGHT.19, S2.P
- net +3V3: now also JUMPER.1
- net BATT_CHECK: now also RIGHT.6; no longer RIGHT.7
- net CHECK_EN: now also R2.1, RIGHT.7; no longer RIGHT.13
- net GND: now also BATT.1, JUMPER.8; no longer C3.2, C5.2, IC2.GND
- net N$7: now also BATT.2, S2.S
- net VCC: now also C1.1, C4.1, DRIVER.CE; no longer C5.1, IC2.+VS, RIGHT.19
