File: Eagle/Micromouse2/Micromouse2.brd (EAGLE design)
At the start: 50.8 x 75.9 mm, 14 parts

Commit message: new schematics
Routing:
- net N$6: track 44.5 -> 79.9 mm
- net GND: track 147.8 -> 130.7 mm
- net N$5: track 64.1 -> 71.2 mm
- net TICK1: track 31.5 -> 36.6 mm
- net N$9: track 12.9 -> 17.8 mm
- net RS_SENS: track 25.6 -> 29.4 mm
- net N$3: track 34.0 -> 36.7 mm
- net RF_SENS: track 25.3 -> 23.3 mm
- net N$8: track 10.3 -> 12.1 mm, vias 1 -> 0
- net N$1: track 32.1 -> 30.4 mm
- net TICK2: track 60.9 -> 62.6 mm
- net LS_SENS: track 34.9 -> 33.4 mm
- net LF_SENS: track 20.2 -> 18.7 mm
- net +3V3: track 103.7 -> 102.3 mm
- net SSENS_EN: track 30.9 -> 32.3 mm
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Other:
- board text added: "* SPARKLES *"
